Commit message: Added gazebo sim to locobot + basic ros_control intf; reverted nav stack param to prv values

File: locobot_description/urdf/camera_head.urdf.xacro (robot description, xacro)
@@ -2,5 +2,12 @@
 <robot name="locobot_camera_head" xmlns:xacro="http://ros.org/wiki/xacro">
     <xacro:include filename="$(find realsense2_description)/urdf/_d435.urdf.xacro"/>
-    <link name="head_link"/>
+    <link name="head_link">
+        <inertial>
+            <mass value="1e-5"/>
+            <inertia ixx="1e-6" ixy="0"    ixz="0"
+                                iyy="1e-6" iyz="0"
+                                           izz="1e-6"/>
+        </inertial>
+    </link>
     <joint name="head_pan_joint" type="revolute">
         <origin xyz="0 0 0" rpy="0 0 0"/>

File: locobot_description/urdf/lds.urdf.xacro (robot description, xacro)
@@ -18,4 +18,11 @@
             </geometry>
         </collision>
+        <inertial>
+            <mass value="1e-5"/>
+            <origin xyz="0 0 0.025" rpy="0 0 0"/>
+            <inertia ixx="1e-6" ixy="0.0"  ixz="0.0"
+                                iyy="1e-6" iyz="0.0"
+                                           izz="1e-6"/>
+        </inertial>
     </link>
     <joint name="scan_joint" type="fixed">

File: locobot_description/urdf/locobot.gazebo.xacro (robot description, xacro)
@@ -1,12 +1,9 @@
 <?xml version="1.0"?>
 <robot name="locobot_sim" xmlns:xacro="http://ros.org/wiki/xacro">
-    <xacro:include filename="$(find kobuki_description)/urdf/kobuki_gazebo.urdf.xacro"/>
-    <xacro:kobuki_sim/>
     <gazebo reference="scan_link">
-        <material>Gazebo/FlatBlack</material>
         <sensor type="ray" name="lds_lfcd_sensor">
             <pose>0 0 0 0 0 0</pose>
-            <visualize>$(arg laser_visual)</visualize>
-            <update_rate>5</update_rate>
+            <visualize>false</visualize>
+            <update_rate>20.0</update_rate>
             <ray>
                 <scan>
@@ -15,5 +12,5 @@
                         <resolution>1</resolution>
                         <min_angle>0.0</min_angle>
-                        <max_angle>6.28319</max_angle>
+                        <max_angle>${2*pi}</max_angle>
                     </horizontal>
                 </scan>
@@ -31,10 +28,12 @@
             <plugin name="gazebo_ros_lds_lfcd_controller" filename="libgazebo_ros_laser.so">
                 <topicName>scan</topicName>
-                <frameName>base_scan</frameName>
+                <frameName>scan_link</frameName>
             </plugin>
         </sensor>
     </gazebo>
     <gazebo>
-        <plugin name="gazebo_ros_control" filename="libgazebo_ros_control.so"/>
+        <plugin name="gazebo_ros_control" filename="libgazebo_ros_control.so">
+            <robotNamespace>/</robotNamespace>
+        </plugin>
     </gazebo>
 </robot>

File: locobot_description/urdf/locobot.urdf.xacro (robot description, xacro)
@@ -82,3 +82,4 @@
     </joint>
     <xacro:include filename="$(find locobot_description)/urdf/camera_head.urdf.xacro"/>
+    <xacro:include filename="$(find locobot_description)/urdf/locobot.gazebo.xacro"/>
 </robot>
